File: pcb 1/Demcare.kicad_sch (KiCad schematic)
At the start: 17 parts, among them J1 USB_B_Micro, J3 Lipo-Bat, SW2 Reset, SW3 Boot, U1 ESP32-WROOM-32, U2 CH340C, U4 TP4057, U5 MIC5504-3.3YM5

Commit message: rerouted the pcb
Parts:
- U4: footprint Package_TO_SOT_SMD:TSOT-23-5 -> Package_TO_SOT_SMD:SOT-23-6
Changed lines of the file:
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@@
 			)
 		)
-		(property "Footprint" "Package_TO_SOT_SMD:TSOT-23-5"
+		(property "Footprint" "Package_TO_SOT_SMD:SOT-23-6"
 			(at 181.61 138.43 0)
 			(effects
